Commit message: maj simu - essai correction coef de frottement

File: src/car_square/model/gazebo.xacro (robot description, xacro)
@@ -1,31 +1,36 @@
 <?xml version="1.0"?>
 <robot xmlns:xacro="http://ros.org/wiki/xacro">
-<gazebo>
+    <gazebo>
         <plugin filename="gz_ros2_control-system" name="gz_ros2_control::GazeboSimROS2ControlPlugin">
-                <parameters>$(find car_square)/config/robot_controller.yaml</parameters>
+            <parameters>$(find car_square)/config/robot_controller.yaml</parameters>
         </plugin>
-</gazebo>
-<gazebo>
-        <plugin
-                filename="gz-sim-sensors-system"
-                name="gz::sim::systems::Sensors">
-                <render_engine>ogre2</render_engine>
+    </gazebo>
+    <gazebo>
+        <plugin filename="gz-sim-sensors-system" name="gz::sim::systems::Sensors">
+            <render_engine>ogre2</render_engine>
         </plugin>
-</gazebo>
-<gazebo reference="lf_hub">
-        <mu1>0.2</mu1>
-        <mu2>0.2</mu2>
-</gazebo>
-<gazebo reference="rf_hub">
-        <mu1>0.2</mu1>
-        <mu2>0.2</mu2>
-</gazebo>
-<gazebo reference="lb_hub">
-        <mu1>0.2</mu1>
-        <mu2>0.2</mu2>
-</gazebo>
-<gazebo reference="rb_hub">
-        <mu1>0.2</mu1>
-        <mu2>0.2</mu2>
-</gazebo>
+    </gazebo>
+    <xacro:property name="friction_coefficient" value="1.0"/>
+    <xacro:property name="num_rollers" value="6"/>
+    <xacro:macro name="set_friction_for_one" params="name">
+        <gazebo reference="${name}">
+                <mu1>${friction_coefficient}</mu1>
+                <mu2>${friction_coefficient}</mu2>
+        </gazebo>
+    </xacro:macro>
+    <xacro:macro name="set_frictions" params="prefix idx">
+        <xacro:if value="${idx &lt; num_rollers}">
+                <xacro:set_friction_for_one name="${prefix}_roller_${idx}"></xacro:set_friction_for_one>
+                <xacro:set_friction_for_one name="${prefix}_roller_neighbor_${idx}"></xacro:set_friction_for_one>
+                <xacro:set_frictions prefix="${prefix}" idx="${idx + 1}" />
+        </xacro:if>
+    </xacro:macro>
+    <xacro:macro name="wheel_friction" params="prefix">
+        <xacro:set_friction_for_one name="${prefix}_hub"></xacro:set_friction_for_one>
+        <xacro:set_frictions prefix="${prefix}" idx="0"/>
+    </xacro:macro>
+    <xacro:wheel_friction prefix="lf"/>
+    <xacro:wheel_friction prefix="rf"/>
+    <xacro:wheel_friction prefix="lb"/>
+    <xacro:wheel_friction prefix="rb"/>
 </robot>

File: src/car_square/model/model_simu.xacro (robot description, xacro)
@@ -1,6 +1,6 @@
 <?xml version="1.0"?>
 <robot name="simple_robot" xmlns:xacro="http://www.ros.org/wiki/xacro">
+        <xacro:include filename="$(find car_square)/model/wheels/omni_wheel.urdf.xacro"/>
         <xacro:include filename="$(find car_square)/model/gazebo.xacro"/>
-        <xacro:include filename="$(find car_square)/model/wheels/omni_wheel.urdf.xacro"/>
         <link name="base_link">
                 <visual>

File: src/car_square/model/parameters.xacro (robot description, xacro)
@@ -24,4 +24,5 @@
 <xacro:property name="roller_length" value="${0.03*SCALE_FACTOR}"/>
 <xacro:property name="roller_count" value="6"/>
+<xacro:property name="friction_coefficient" value="100"/>
 <material name="blue">
         <color rgba="0 0 1 1"/>

Commit message: Rajout d'un lidar dans la simu

File: src/car_square/model/gazebo.xacro (robot description, xacro)
@@ -4,9 +4,4 @@
         <plugin filename="gz_ros2_control-system" name="gz_ros2_control::GazeboSimROS2ControlPlugin">
             <parameters>$(find car_square)/config/robot_controller.yaml</parameters>
-        </plugin>
-    </gazebo>
-    <gazebo>
-        <plugin filename="gz-sim-sensors-system" name="gz::sim::systems::Sensors">
-            <render_engine>ogre2</render_engine>
         </plugin>
     </gazebo>
@@ -34,3 +29,38 @@
     <xacro:wheel_friction prefix="lb"/>
     <xacro:wheel_friction prefix="rb"/>
+    <!-- LIDAR SENSOR -->
+    <gazebo>
+        <plugin filename="gz-sim-sensors-system" name="gz::sim::systems::Sensors">
+            <render_engine>ogre2</render_engine>
+        </plugin>
+    </gazebo>
+    <gazebo reference="lidar_link">
+        <sensor name="gpu_lidar" type="gpu_lidar">
+            <pose relative_to="lidar_link">0 0 0 0 0 0</pose>
+            <topic>scan</topic>
+            <update_rate>2</update_rate>
+            <lidar>
+                <scan>
+                    <horizontal>
+                        <samples>720</samples>
+                        <resolution>1</resolution>
+                        <min_angle>-3.14</min_angle>
+                        <max_angle>3.14</max_angle>
+                    </horizontal>
+                </scan>
+                <range>
+                    <min>0.01</min>
+                    <max>12.0</max>
+                    <resolution>0.005</resolution>
+                </range>
+                <noise>
+                    <type>gaussian</type>
+                    <mean>0.0</mean>
+                    <stddev>0.001</stddev>
+                </noise>
+            </lidar>
+            <always_on>1</always_on>
+            <visualize>1</visualize>
+        </sensor>
+    </gazebo>
 </robot>

File: src/car_square/model/model_simu.xacro (robot description, xacro)
@@ -24,5 +24,5 @@
                         <box size="${chassis_length/8} ${chassis_width/2} ${chassis_height/4}"/>
                         </geometry>
-                        <origin xyz="${3*chassis_length/8} 0 ${1.5*chassis_offset - chassis_height/8}" rpy="0 0 0"/>
+                        <origin xyz="0 0 0" rpy="0 0 0"/>
                         <material name="green"/>
                 </visual>
@@ -31,5 +31,5 @@
                 <parent link="base_link"/>
                 <child link="visual_front"/>
-                <origin xyz="0 0 0" rpy="0 0 0"/>
+                <origin xyz="${3*chassis_length/8} 0 ${1.5*chassis_offset - chassis_height/8}" rpy="0 0 0"/>
         </joint>
         <!-- LINKS ET JOINTS DES ROUES -->
@@ -58,4 +58,31 @@
                 rpy="0 0 ${-5*pi/4}"
         />
+        <link name="lidar_link">
+                <visual>
+                        <origin xyz="0 0 0" rpy="0 0 0"/>
+                        <geometry>
+                                <cylinder length="0.1" radius="0.1"/>
+                        </geometry>
+                </visual>
+                <collision name="collision">
+                        <origin xyz="0 0 0" rpy="0 0 0"/>
+                        <geometry>
+                                <cylinder length="0.1" radius="0.1"/>
+                        </geometry>
+                </collision>
+                <inertial>
+                        <mass value="1e-6"/>
+                        <origin xyz="0 0 0" rpy="0 0 0"/>
+                        <inertia ixx="1e-6" ixy="0" ixz="0"
+                                 iyy="1e-6" iyz="0" izz="1e-6"
+                        />
+                </inertial>
+        </link>
+        <joint name="lidar_joint" type="fixed">
+                        <origin xyz="0 0 ${2*chassis_offset - chassis_height/8}" rpy="0 0 0"/>
+                <parent link="base_link"/>
+                <child link="lidar_link"/>
+                <axis xyz="0 1 0" rpy="0 0 0"/>
+        </joint>
         <!-- ROS2_CONTROL -->
         <ros2_control name="RobotController" type="system">

File: src/car_square/model/wheels/omni_wheel.urdf.xacro (robot description, xacro)
@@ -6,6 +6,6 @@
     <link name="${prefix}_roller_${idx}">
       <inertial>
-        <origin xyz="0 0 0"/>
-        <mass value="0.02"/>
+        <origin rpy="1.5708 0 0"/>
+        <mass value="5"/>
         <inertia
           ixx="0.00001" iyy="0.00001" izz="0.00001"
@@ -28,6 +28,6 @@
     <link name="${prefix}_roller_neighbor_${idx}">
       <inertial>
-        <origin xyz="0 0 0"/>
-        <mass value="0.02"/>
+        <origin rpy="1.5708 0 0"/>
+        <mass value="5"/>
         <inertia
           ixx="0.00001" iyy="0.00001" izz="0.00001"
@@ -55,4 +55,5 @@
         rpy="${3*pi/2 - angle1} 0 1.5708"/>
       <axis xyz="0 1 0"/>
+      <dynamics damping="100.0" friction="5.0"/>
     </joint>
     <joint name="${prefix}_roller_neighbor_${idx}_joint" type="continuous">
@@ -63,4 +64,5 @@
         rpy="${3*pi/2 - angle2} 0 1.5708"/>
       <axis xyz="0 1 0"/>
+      <dynamics damping="100.0" friction="5.0"/>
     </joint>
   </xacro:macro>
@@ -101,5 +103,5 @@
     <link name="${prefix}_hub">
       <inertial>
-        <origin xyz="0 0 0"/>
+        <origin rpy="1.5708 0 0"/>
         <mass value="0.5"/>
         <inertia
@@ -127,4 +129,5 @@
       <origin xyz="${xyz}" rpy="${rpy}"/>
       <axis xyz="0 1 0"/>
+      <dynamics damping="100.0" friction="5.0"/>
     </joint>
     <!-- génération des rollers -->
