Commit message: Changement des roues -> fichiers stl importés

File: src/car_square/model/gazebo.xacro (robot description, xacro)
@@ -6,27 +6,4 @@
         </plugin>
     </gazebo>
-    <xacro:property name="friction_coefficient" value="1.0"/>
-    <xacro:property name="num_rollers" value="6"/>
-    <xacro:macro name="set_friction_for_one" params="name">
-        <gazebo reference="${name}">
-                <mu1>${friction_coefficient}</mu1>
-                <mu2>${friction_coefficient}</mu2>
-        </gazebo>
-    </xacro:macro>
-    <xacro:macro name="set_frictions" params="prefix idx">
-        <xacro:if value="${idx &lt; num_rollers}">
-                <xacro:set_friction_for_one name="${prefix}_roller_${idx}"></xacro:set_friction_for_one>
-                <xacro:set_friction_for_one name="${prefix}_roller_neighbor_${idx}"></xacro:set_friction_for_one>
-                <xacro:set_frictions prefix="${prefix}" idx="${idx + 1}" />
-        </xacro:if>
-    </xacro:macro>
-    <xacro:macro name="wheel_friction" params="prefix">
-        <xacro:set_friction_for_one name="${prefix}_hub"></xacro:set_friction_for_one>
-        <xacro:set_frictions prefix="${prefix}" idx="0"/>
-    </xacro:macro>
-    <xacro:wheel_friction prefix="lf"/>
-    <xacro:wheel_friction prefix="rf"/>
-    <xacro:wheel_friction prefix="lb"/>
-    <xacro:wheel_friction prefix="rb"/>
     <!-- LIDAR SENSOR -->
     <gazebo>
@@ -36,8 +13,9 @@
     </gazebo>
     <gazebo reference="lidar_link">
-        <sensor name="gpu_lidar" type="gpu_lidar">
+        <sensor name="lidar" type="gpu_lidar">
             <pose relative_to="lidar_link">0 0 0 0 0 0</pose>
             <topic>scan</topic>
-            <update_rate>2</update_rate>
+            <update_rate>10</update_rate>
+            <gz_frame_id>lidar_link</gz_frame_id>
             <lidar>
                 <scan>
@@ -57,5 +35,5 @@
                     <type>gaussian</type>
                     <mean>0.0</mean>
-                    <stddev>0.001</stddev>
+                    <stddev>0.01</stddev>
                 </noise>
             </lidar>

File: src/car_square/model/model_simu.xacro (robot description, xacro)
@@ -31,5 +31,5 @@
                 <parent link="base_link"/>
                 <child link="visual_front"/>
-                <origin xyz="${3*chassis_length/8} 0 ${1.5*chassis_offset - chassis_height/8}" rpy="0 0 0"/>
+                <origin xyz="${chassis_length/2} 0 ${chassis_offset}" rpy="0 1.571 0"/>
         </joint>
         <!-- LINKS ET JOINTS DES ROUES -->
@@ -58,27 +58,44 @@
                 rpy="0 0 ${-5*pi/4}"
         />
+        <!--  -->
+        <link name="mat_link">
+                <visual>
+                        <origin xyz="0 0 0" rpy="0 0 0"/>
+                        <geometry>
+                                <cylinder length="${mat_length}" radius="${mat_radius}"/>
+                        </geometry>
+                        <material name="red"/>
+                </visual>
+                <collision name="collision">
+                        <origin xyz="0 0 0" rpy="0 0 0"/>
+                        <geometry>
+                                <cylinder length="${mat_length}" radius="${mat_radius}"/>
+                        </geometry>
+                </collision>
+        </link>
+        <joint name="mat_joint" type="fixed">
+                        <origin xyz="0 0 ${chassis_offset - chassis_height/4 + mat_length/2}" rpy="0 0 0"/>
+                <parent link="base_link"/>
+                <child link="mat_link"/>
+                <axis xyz="0 1 0" rpy="0 0 0"/>
+        </joint>
+        <!-- LINKS ET JOINTS DU LIDAR -->
         <link name="lidar_link">
                 <visual>
                         <origin xyz="0 0 0" rpy="0 0 0"/>
                         <geometry>
-                                <cylinder length="0.1" radius="0.1"/>
+                                <cylinder length="${lidar_length}" radius="${lidar_radius}"/>
                         </geometry>
+                        <material name="green"/>
                 </visual>
                 <collision name="collision">
                         <origin xyz="0 0 0" rpy="0 0 0"/>
                         <geometry>
-                                <cylinder length="0.1" radius="0.1"/>
+                                <cylinder length="${lidar_length}" radius="${lidar_radius}"/>
                         </geometry>
                 </collision>
-                <inertial>
-                        <mass value="1e-6"/>
-                        <origin xyz="0 0 0" rpy="0 0 0"/>
-                        <inertia ixx="1e-6" ixy="0" ixz="0"
-                                 iyy="1e-6" iyz="0" izz="1e-6"
-                        />
-                </inertial>
         </link>
         <joint name="lidar_joint" type="fixed">
-                        <origin xyz="0 0 ${2*chassis_offset - chassis_height/8}" rpy="0 0 0"/>
+                        <origin xyz="0 0 ${chassis_offset - chassis_height/4 + mat_length + lidar_length/2}" rpy="0 0 0"/>
                 <parent link="base_link"/>
                 <child link="lidar_link"/>

File: src/car_square/model/parameters.xacro (robot description, xacro)
@@ -19,10 +19,13 @@
 </xacro:macro>
 <xacro:property name="r" value="${0.1*SCALE_FACTOR}" />
-<xacro:property name="wheel_radius" value="${0.06*SCALE_FACTOR}"/>
-<xacro:property name="wheel_width" value="${0.02*SCALE_FACTOR}"/>
+<xacro:property name="wheel_radius" value="${0.065*SCALE_FACTOR}"/>
+<xacro:property name="wheel_width" value="${0.03*SCALE_FACTOR}"/>
 <xacro:property name="roller_radius" value="${0.01*SCALE_FACTOR}"/>
 <xacro:property name="roller_length" value="${0.03*SCALE_FACTOR}"/>
-<xacro:property name="roller_count" value="6"/>
-<xacro:property name="friction_coefficient" value="100"/>
+<xacro:property name="roller_count" value="4"/>
+<xacro:property name="mat_radius" value="${0.2*SCALE_FACTOR}"/>
+<xacro:property name="mat_length" value="${0.6*SCALE_FACTOR}"/>
+<xacro:property name="lidar_radius" value="${0.02*SCALE_FACTOR}"/>
+<xacro:property name="lidar_length" value="${0.02*SCALE_FACTOR}"/>
 <material name="blue">
         <color rgba="0 0 1 1"/>

File: src/car_square/model/wheels/omni_wheel.urdf.xacro (robot description, xacro)
@@ -6,46 +6,76 @@
     <link name="${prefix}_roller_${idx}">
       <inertial>
-        <origin rpy="1.5708 0 0"/>
-        <mass value="5"/>
-        <inertia
-          ixx="0.00001" iyy="0.00001" izz="0.00001"
-          ixy="0" ixz="0" iyz="0"/>
+        <mass value="9.1"/>
+        <inertia ixx="0.0812" iyy="0.0812" izz="0.0473" ixy="0" ixz="0" iyz="0"/>
       </inertial>
       <collision>
-        <origin rpy="1.5708 0 0"/>
+        <origin xyz="0 0 0" rpy="1.571 0 0"/>
         <geometry>
-          <cylinder radius="${roller_radius}" length="${roller_length}"/>
+          <mesh filename="file://$(find car_square)/meshes/roller.stl" scale="${wheel_radius*61.5384615385} ${wheel_radius*61.5384615385} ${wheel_radius*61.5384615385}"/>
         </geometry>
       </collision>
       <visual>
-        <origin rpy="1.5708 0 0"/>
+        <origin xyz="0 0 0" rpy="1.571 0 0"/>
         <geometry>
-          <cylinder radius="${roller_radius}" length="${roller_length}"/>
+          <mesh filename="file://$(find car_square)/meshes/roller.stl" scale="${wheel_radius*61.5384615385} ${wheel_radius*61.5384615385} ${wheel_radius*61.5384615385}"/>
         </geometry>
-        <material name="white" />
+        <material name="white"/>
       </visual>
     </link>
+    <gazebo reference="${prefix}_roller_${idx}">
+      <surface>
+        <friction>
+          <ode>
+            <mu>1.0</mu>
+            <mu2>1.0</mu2>
+          </ode>
+        </friction>
+        <contact>
+          <ode>
+            <kp>1e+5</kp>
+            <kd>100.0</kd>
+            <max_vel>0.01</max_vel>
+            <min_depth>0</min_depth>
+          </ode>
+        </contact>
+      </surface>
+    </gazebo>
     <link name="${prefix}_roller_neighbor_${idx}">
       <inertial>
-        <origin rpy="1.5708 0 0"/>
-        <mass value="5"/>
-        <inertia
-          ixx="0.00001" iyy="0.00001" izz="0.00001"
-          ixy="0" ixz="0" iyz="0"/>
+        <mass value="9.1"/>
+        <inertia ixx="0.0812" iyy="0.0812" izz="0.0473" ixy="0" ixz="0" iyz="0"/>
       </inertial>
       <collision>
-        <origin rpy="1.5708 0 0"/>
+        <origin xyz="0 0 0" rpy="1.571 0 0"/>
         <geometry>
-          <cylinder radius="${roller_radius}" length="${roller_length}"/>
+          <mesh filename="file://$(find car_square)/meshes/roller.stl" scale="${wheel_radius*61.5384615385} ${wheel_radius*61.5384615385} ${wheel_radius*61.5384615385}"/>
         </geometry>
       </collision>
       <visual>
-        <origin rpy="1.5708 0 0"/>
+        <origin xyz="0 0 0" rpy="1.571 0 0"/>
         <geometry>
-          <cylinder radius="${roller_radius}" length="${roller_length}"/>
+          <mesh filename="file://$(find car_square)/meshes/roller.stl" scale="${wheel_radius*61.5384615385} ${wheel_radius*61.5384615385} ${wheel_radius*61.5384615385}"/>
         </geometry>
-        <material name="white" />
+        <material name="white"/>
       </visual>
     </link>
+    <gazebo reference="${prefix}_roller_neighbor_${idx}">
+      <surface>
+        <friction>
+          <ode>
+            <mu>1.0</mu>
+            <mu2>1.0</mu2>
+          </ode>
+        </friction>
+        <contact>
+          <ode>
+            <kp>1e+5</kp>
+            <kd>100.0</kd>
+            <max_vel>0.01</max_vel>
+            <min_depth>0</min_depth>
+          </ode>
+        </contact>
+      </surface>
+    </gazebo>
     <joint name="${prefix}_roller_${idx}_joint" type="continuous">
       <parent link="${parent}"/>
@@ -55,5 +85,5 @@
         rpy="${3*pi/2 - angle1} 0 1.5708"/>
       <axis xyz="0 1 0"/>
-      <dynamics damping="100.0" friction="5.0"/>
+      <dynamics damping="0.01" friction="0.0"/>
     </joint>
     <joint name="${prefix}_roller_neighbor_${idx}_joint" type="continuous">
@@ -61,8 +91,8 @@
       <child link="${prefix}_roller_neighbor_${idx}"/>
       <origin
-        xyz="${(wheel_radius - roller_radius) * cos(angle2)} ${2*roller_radius - wheel_width/2} ${(wheel_radius - roller_radius) * sin(angle2)}"
+        xyz="${(wheel_radius - roller_radius) * cos(angle2)} ${wheel_width/2} ${(wheel_radius - roller_radius) * sin(angle2)}"
         rpy="${3*pi/2 - angle2} 0 1.5708"/>
       <axis xyz="0 1 0"/>
-      <dynamics damping="100.0" friction="5.0"/>
+      <dynamics damping="0.01" friction="0.0"/>
     </joint>
   </xacro:macro>
@@ -71,57 +101,58 @@
                params="prefix parent idx count wheel_radius wheel_width roller_radius roller_length">
     <xacro:if value="${idx &lt; count}">
-      <xacro:property name="angle1"
-                      value="${2 * pi * idx / count}"/>
-      <xacro:property name="angle2"
-                      value="${2 * pi * idx / count + pi / count}" />
+      <xacro:property name="angle1" value="${2 * pi * idx / count}"/>
+      <xacro:property name="angle2" value="${2 * pi * idx / count + pi / count}"/>
       <xacro:roller
-        prefix="${prefix}"
-        parent="${parent}"
-        idx="${idx}"
-        angle1="${angle1}"
-        angle2="${angle2}"
-        wheel_radius="${wheel_radius}"
-        wheel_width="${wheel_width}"
-        roller_radius="${roller_radius}"
-        roller_length="${roller_length}"/>
-      <!-- appel récursif -->
+        prefix="${prefix}" parent="${parent}" idx="${idx}"
+        angle1="${angle1}" angle2="${angle2}"
+        wheel_radius="${wheel_radius}" wheel_width="${wheel_width}"
+        roller_radius="${roller_radius}" roller_length="${roller_length}"/>
       <xacro:roller_loop
-        prefix="${prefix}"
-        parent="${parent}"
-        idx="${idx + 1}"
-        count="${count}"
-        wheel_radius="${wheel_radius}"
-        wheel_width="${wheel_width}"
-        roller_radius="${roller_radius}"
-        roller_length="${roller_length}"/>
+        prefix="${prefix}" parent="${parent}" idx="${idx + 1}" count="${count}"
+        wheel_radius="${wheel_radius}" wheel_width="${wheel_width}"
+        roller_radius="${roller_radius}" roller_length="${roller_length}"/>
     </xacro:if>
   </xacro:macro>
   <!-- ========== OMNI WHEEL COMPLETE ========== -->
-  <xacro:macro name="omni_wheel"
-               params="prefix parent xyz rpy">
-    <!-- moyeu -->
+  <xacro:macro name="omni_wheel" params="prefix parent xyz rpy">
     <link name="${prefix}_hub">
       <inertial>
         <origin rpy="1.5708 0 0"/>
-        <mass value="0.5"/>
-        <inertia
-          ixx="0.001" iyy="0.001" izz="0.001"
-          ixy="0.0" ixz="0.0" iyz="0.0"/>
+        <mass value="66.86064"/>
+        <inertia ixx="3.009" iyy="2.1239" izz="2.1239" ixy="0.0" ixz="0.0" iyz="0.0"/>
       </inertial>
       <visual>
+        <origin xyz="0 0 0" rpy="0 0 1.571"/>
         <geometry>
-          <cylinder radius="${7*wheel_radius/8}" length="${3*wheel_width/2}"/>
+          <mesh filename="file://$(find car_square)/meshes/rim.stl" scale="${wheel_radius*61.5384615385} ${wheel_radius*61.5384615385} ${wheel_radius*61.5384615385}"/>
         </geometry>
         <material name="blue"/>
-        <origin rpy="1.5708 0 0"/>
       </visual>
       <collision>
+        <origin xyz="0 0 0" rpy="0 0 1.571"/>
         <geometry>
-          <cylinder radius="${7*wheel_radius/8}" length="${3*wheel_width/2}"/>
+          <mesh filename="file://$(find car_square)/meshes/rim.stl" scale="${wheel_radius*61.5384615385} ${wheel_radius*61.5384615385} ${wheel_radius*61.5384615385}"/>
         </geometry>
-        <material name="blue"/>
-        <origin rpy="1.5708 0 0"/>
       </collision>
     </link>
+    <gazebo reference="${prefix}_hub">
+      <surface>
+        <friction>
+          <ode>
+            <mu>1.0</mu>
+            <mu2>1.0</mu2>
+            <fdir1>0 0 0</fdir1>
+          </ode>
+        </friction>
+        <contact>
+          <ode>
+            <kp>1e+5</kp>
+            <kd>100.0</kd>
+            <max_vel>0.01</max_vel>
+            <min_depth>0</min_depth>
+          </ode>
+        </contact>
+      </surface>
+    </gazebo>
     <joint name="${prefix}_joint" type="continuous">
       <parent link="${parent}"/>
@@ -129,16 +160,11 @@
       <origin xyz="${xyz}" rpy="${rpy}"/>
       <axis xyz="0 1 0"/>
-      <dynamics damping="100.0" friction="5.0"/>
+      <dynamics damping="0.0" friction="0.0"/>
     </joint>
-    <!-- génération des rollers -->
     <xacro:roller_loop
-      prefix="${prefix}"
-      parent="${prefix}_hub"
-      idx="0"
-      count="${roller_count}"
-      wheel_radius="${wheel_radius}"
-      wheel_width="${wheel_width}"
-      roller_radius="${roller_radius}"
-      roller_length="${roller_length}"/>
+      prefix="${prefix}" parent="${prefix}_hub"
+      idx="0" count="${roller_count}"
+      wheel_radius="${wheel_radius}" wheel_width="${wheel_width}"
+      roller_radius="${roller_radius}" roller_length="${roller_length}"/>
   </xacro:macro>
 </robot>
