Commit message: Ajout d'un paramètre d'accération

File: src/car_square/model/model_simu.xacro (robot description, xacro)
@@ -37,5 +37,5 @@
                 prefix="lf"
                 parent="base_link"
-                xyz="${chassis_length/2} ${chassis_width/2 + wheel_width} ${r}"
+                xyz="${chassis_length/2} ${chassis_width/2} ${r}"
                 rpy="0 0 ${-pi/4}"
         />
@@ -43,5 +43,5 @@
                 prefix="rf"
                 parent="base_link"
-                xyz="${chassis_length/2} ${-(chassis_width/2 + wheel_width)} ${r}"
+                xyz="${chassis_length/2} ${-(chassis_width/2)} ${r}"
                 rpy="0 0 ${5*pi/4}"
         />
@@ -49,5 +49,5 @@
                 prefix="lb"
                 parent="base_link"
-                xyz="${-(chassis_length/2)} ${chassis_width/2 + wheel_width} ${r}"
+                xyz="${-(chassis_length/2)} ${chassis_width/2} ${r}"
                 rpy="0 0 ${pi/4}"
         />
@@ -55,5 +55,5 @@
                 prefix="rb"
                 parent="base_link"
-                xyz="${-(chassis_length/2)} ${-(chassis_width/2 + wheel_width)} ${r}"
+                xyz="${-(chassis_length/2)} ${-(chassis_width/2)} ${r}"
                 rpy="0 0 ${-5*pi/4}"
         />

File: src/car_square/model/wheels/omni_wheel.urdf.xacro (robot description, xacro)
@@ -6,6 +6,6 @@
     <link name="${prefix}_roller_${idx}">
       <inertial>
-        <mass value="0.1"/>
-        <inertia ixx="10" iyy="10" izz="10" ixy="0" ixz="0" iyz="0"/>
+        <mass value="0.02"/>
+        <inertia ixx="1e-6" iyy="1e-6" izz="1e-6" iyz="0" ixy="0" ixz="0"/>
       </inertial>
       <collision>
@@ -24,16 +24,16 @@
     </link>
     <gazebo reference="${prefix}_roller_${idx}">
-      <mu>1</mu>
-      <mu2>1</mu2>
+      <mu>5</mu>
+      <mu2>5</mu2>
       <slip1>0</slip1>
       <slip2>0</slip2>
-      <kp>1e+13</kp>  <!-- Rigidité très élevée -->
-      <kd>1.0</kd>
+      <kp>5e5</kp>
+      <kd>50</kd>
       <material>Gazebo/Grey</material>
     </gazebo>
     <link name="${prefix}_roller_neighbor_${idx}">
       <inertial>
-        <mass value="0.1"/>
-        <inertia ixx="10" iyy="10" izz="10" ixy="0" ixz="0" iyz="0"/>
+        <mass value="0.02"/>
+        <inertia ixx="1e-6" iyy="1e-6" izz="1e-6" iyz="0" ixy="0" ixz="0"/>
       </inertial>
       <collision>
@@ -52,10 +52,10 @@
     </link>
     <gazebo reference="${prefix}_roller_neighbor_${idx}">
-      <mu>1</mu>
-      <mu2>1</mu2>
+      <mu>5</mu>
+      <mu2>5</mu2>
       <slip1>0</slip1>
       <slip2>0</slip2>
-      <kp>1e+13</kp>  <!-- Rigidité très élevée -->
-      <kd>1.0</kd>
+      <kp>5e5</kp>
+      <kd>50</kd>
       <material>Gazebo/Grey</material>
     </gazebo>
@@ -67,5 +67,5 @@
         rpy="${3*pi/2 - angle1} 0 1.5708"/>
       <axis xyz="0 1 0"/>
-      <dynamics damping="0.0" friction="0.0"/>
+      <dynamics damping="5.0" friction="1.0"/>
     </joint>
     <joint name="${prefix}_roller_neighbor_${idx}_joint" type="continuous">
@@ -76,5 +76,5 @@
         rpy="${3*pi/2 - angle2} 0 1.5708"/>
       <axis xyz="0 1 0"/>
-      <dynamics damping="0.0" friction="0.0"/>
+      <dynamics damping="5.0" friction="1.0"/>
     </joint>
   </xacro:macro>
@@ -101,6 +101,6 @@
       <inertial>
         <origin rpy="1.5708 0 0"/>
-        <mass value="66.86064"/>
-        <inertia ixx="0.009" iyy="0.1239" izz="0.1239" ixy="0.0" ixz="0.0" iyz="0.0"/>
+        <mass value="1.0"/>
+        <inertia ixx="0.0001" iyy="0.0001" izz="0.0001" ixy="0" ixz="0" iyz="0"/>
       </inertial>
       <visual>
@@ -129,6 +129,6 @@
         <contact>
           <ode>
-            <kp>1e+6</kp>
-            <kd>100.0</kd>
+            <kp>5e5</kp>
+            <kd>50</kd>
             <max_vel>0.01</max_vel>
             <min_depth>0.001</min_depth>
@@ -142,5 +142,5 @@
       <origin xyz="${xyz}" rpy="${rpy}"/>
       <axis xyz="0 1 0"/>
-      <dynamics damping="0.5" friction="0.1"/>
+      <dynamics damping="1.0" friction="0.5"/>
     </joint>
     <xacro:roller_loop

Commit message: maj

File: src/car_square/model/model_simu.xacro (robot description, xacro)
@@ -22,5 +22,5 @@
                 <visual>
                         <geometry>
-                        <box size="${chassis_length/8} ${chassis_width/2} ${chassis_height/4}"/>
+                                <box size="${chassis_length/8} ${chassis_width/2} ${chassis_height/4}"/>
                         </geometry>
                         <origin xyz="0 0 0" rpy="0 0 0"/>
@@ -37,5 +37,5 @@
                 prefix="lf"
                 parent="base_link"
-                xyz="${chassis_length/2} ${chassis_width/2} ${r}"
+                xyz="${chassis_length/2 + wheel_offset} ${chassis_width/2 + wheel_offset} ${r}"
                 rpy="0 0 ${-pi/4}"
         />
@@ -43,5 +43,5 @@
                 prefix="rf"
                 parent="base_link"
-                xyz="${chassis_length/2} ${-(chassis_width/2)} ${r}"
+                xyz="${chassis_length/2 + wheel_offset} ${-(chassis_width/2 + wheel_offset)} ${r}"
                 rpy="0 0 ${5*pi/4}"
         />
@@ -49,5 +49,5 @@
                 prefix="lb"
                 parent="base_link"
-                xyz="${-(chassis_length/2)} ${chassis_width/2} ${r}"
+                xyz="${-(chassis_length/2 + wheel_offset)} ${chassis_width/2 + wheel_offset} ${r}"
                 rpy="0 0 ${pi/4}"
         />
@@ -55,5 +55,5 @@
                 prefix="rb"
                 parent="base_link"
-                xyz="${-(chassis_length/2)} ${-(chassis_width/2)} ${r}"
+                xyz="${-(chassis_length/2 + wheel_offset)} ${-(chassis_width/2 + wheel_offset)} ${r}"
                 rpy="0 0 ${-5*pi/4}"
         />
@@ -112,4 +112,44 @@
                         <state_interface name="velocity"/>
                 </joint>
+                <joint name="lf_roller_0_joint">
+                        <command_interface name="velocity"/>
+                        <state_interface name="position"/>
+                        <state_interface name="velocity"/>
+                </joint>
+                <joint name="lf_roller_neighbor_0_joint">
+                        <command_interface name="velocity"/>
+                        <state_interface name="position"/>
+                        <state_interface name="velocity"/>
+                </joint>
+                <joint name="lf_roller_1_joint">
+                        <command_interface name="velocity"/>
+                        <state_interface name="position"/>
+                        <state_interface name="velocity"/>
+                </joint>
+                <joint name="lf_roller_neighbor_1_joint">
+                        <command_interface name="velocity"/>
+                        <state_interface name="position"/>
+                        <state_interface name="velocity"/>
+                </joint>
+                <joint name="lf_roller_2_joint">
+                        <command_interface name="velocity"/>
+                        <state_interface name="position"/>
+                        <state_interface name="velocity"/>
+                </joint>
+                <joint name="lf_roller_neighbor_2_joint">
+                        <command_interface name="velocity"/>
+                        <state_interface name="position"/>
+                        <state_interface name="velocity"/>
+                </joint>
+                <joint name="lf_roller_3_joint">
+                        <command_interface name="velocity"/>
+                        <state_interface name="position"/>
+                        <state_interface name="velocity"/>
+                </joint>
+                <joint name="lf_roller_neighbor_3_joint">
+                        <command_interface name="velocity"/>
+                        <state_interface name="position"/>
+                        <state_interface name="velocity"/>
+                </joint>
                 <joint name="rf_joint">
                         <command_interface name="velocity"/>
@@ -117,4 +157,44 @@
                         <state_interface name="velocity"/>
                 </joint>
+                <joint name="rf_roller_0_joint">
+                        <command_interface name="velocity"/>
+                        <state_interface name="position"/>
+                        <state_interface name="velocity"/>
+                </joint>
+                <joint name="rf_roller_neighbor_0_joint">
+                        <command_interface name="velocity"/>
+                        <state_interface name="position"/>
+                        <state_interface name="velocity"/>
+                </joint>
+                <joint name="rf_roller_1_joint">
+                        <command_interface name="velocity"/>
+                        <state_interface name="position"/>
+                        <state_interface name="velocity"/>
+                </joint>
+                <joint name="rf_roller_neighbor_1_joint">
+                        <command_interface name="velocity"/>
+                        <state_interface name="position"/>
+                        <state_interface name="velocity"/>
+                </joint>
+                <joint name="rf_roller_2_joint">
+                        <command_interface name="velocity"/>
+                        <state_interface name="position"/>
+                        <state_interface name="velocity"/>
+                </joint>
+                <joint name="rf_roller_neighbor_2_joint">
+                        <command_interface name="velocity"/>
+                        <state_interface name="position"/>
+                        <state_interface name="velocity"/>
+                </joint>
+                <joint name="rf_roller_3_joint">
+                        <command_interface name="velocity"/>
+                        <state_interface name="position"/>
+                        <state_interface name="velocity"/>
+                </joint>
+                <joint name="rf_roller_neighbor_3_joint">
+                        <command_interface name="velocity"/>
+                        <state_interface name="position"/>
+                        <state_interface name="velocity"/>
+                </joint>
                 <joint name="lb_joint">
                         <command_interface name="velocity"/>
@@ -122,5 +202,85 @@
                         <state_interface name="velocity"/>
                 </joint>
+                <joint name="lb_roller_0_joint">
+                        <command_interface name="velocity"/>
+                        <state_interface name="position"/>
+                        <state_interface name="velocity"/>
+                </joint>
+                <joint name="lb_roller_neighbor_0_joint">
+                        <command_interface name="velocity"/>
+                        <state_interface name="position"/>
+                        <state_interface name="velocity"/>
+                </joint>
+                <joint name="lb_roller_1_joint">
+                        <command_interface name="velocity"/>
+                        <state_interface name="position"/>
+                        <state_interface name="velocity"/>
+                </joint>
+                <joint name="lb_roller_neighbor_1_joint">
+                        <command_interface name="velocity"/>
+                        <state_interface name="position"/>
+                        <state_interface name="velocity"/>
+                </joint>
+                <joint name="lb_roller_2_joint">
+                        <command_interface name="velocity"/>
+                        <state_interface name="position"/>
+                        <state_interface name="velocity"/>
+                </joint>
+                <joint name="lb_roller_neighbor_2_joint">
+                        <command_interface name="velocity"/>
+                        <state_interface name="position"/>
+                        <state_interface name="velocity"/>
+                </joint>
+                <joint name="lb_roller_3_joint">
+                        <command_interface name="velocity"/>
+                        <state_interface name="position"/>
+                        <state_interface name="velocity"/>
+                </joint>
+                <joint name="lb_roller_neighbor_3_joint">
+                        <command_interface name="velocity"/>
+                        <state_interface name="position"/>
+                        <state_interface name="velocity"/>
+                </joint>
                 <joint name="rb_joint">
+                        <command_interface name="velocity"/>
+                        <state_interface name="position"/>
+                        <state_interface name="velocity"/>
+                </joint>
+                <joint name="rb_roller_0_joint">
+                        <command_interface name="velocity"/>
+                        <state_interface name="position"/>
+                        <state_interface name="velocity"/>
+                </joint>
+                <joint name="rb_roller_neighbor_0_joint">
+                        <command_interface name="velocity"/>
+                        <state_interface name="position"/>
+                        <state_interface name="velocity"/>
+                </joint>
+                <joint name="rb_roller_1_joint">
+                        <command_interface name="velocity"/>
+                        <state_interface name="position"/>
+                        <state_interface name="velocity"/>
+                </joint>
+                <joint name="rb_roller_neighbor_1_joint">
+                        <command_interface name="velocity"/>
+                        <state_interface name="position"/>
+                        <state_interface name="velocity"/>
+                </joint>
+                <joint name="rb_roller_2_joint">
+                        <command_interface name="velocity"/>
+                        <state_interface name="position"/>
+                        <state_interface name="velocity"/>
+                </joint>
+                <joint name="rb_roller_neighbor_2_joint">
+                        <command_interface name="velocity"/>
+                        <state_interface name="position"/>
+                        <state_interface name="velocity"/>
+                </joint>
+                <joint name="rb_roller_3_joint">
+                        <command_interface name="velocity"/>
+                        <state_interface name="position"/>
+                        <state_interface name="velocity"/>
+                </joint>
+                <joint name="rb_roller_neighbor_3_joint">
                         <command_interface name="velocity"/>
                         <state_interface name="position"/>

File: src/car_square/model/parameters.xacro (robot description, xacro)
@@ -6,4 +6,5 @@
 <xacro:property name="chassis_height" value="${0.1*SCALE_FACTOR}" />
 <xacro:property name="chassis_offset" value="${0.15*SCALE_FACTOR}" />
+<xacro:property name="wheel_offset" value="${0.04*SCALE_FACTOR}" />
 <xacro:property name="chassis_density" value="271.0"/>
 <xacro:property name="chassis_mass" value="${chassis_density * (chassis_length * chassis_width * chassis_height)}"/>

File: src/car_square/model/wheels/omni_wheel.urdf.xacro (robot description, xacro)
@@ -14,4 +14,5 @@
           <mesh filename="file://$(find car_square)/meshes/roller.stl" scale="${wheel_radius*61.5384615385} ${wheel_radius*61.5384615385} ${wheel_radius*61.5384615385}"/>
         </geometry>
+        <contact_coefficients mu="1.0" kp="0.0" kd="1000.0" />
       </collision>
       <visual>
@@ -23,13 +24,4 @@
       </visual>
     </link>
-    <gazebo reference="${prefix}_roller_${idx}">
-      <mu>5</mu>
-      <mu2>5</mu2>
-      <slip1>0</slip1>
-      <slip2>0</slip2>
-      <kp>5e5</kp>
-      <kd>50</kd>
-      <material>Gazebo/Grey</material>
-    </gazebo>
     <link name="${prefix}_roller_neighbor_${idx}">
       <inertial>
@@ -42,4 +34,5 @@
           <mesh filename="file://$(find car_square)/meshes/roller.stl" scale="${wheel_radius*61.5384615385} ${wheel_radius*61.5384615385} ${wheel_radius*61.5384615385}"/>
         </geometry>
+        <contact_coefficients mu="1.0" kp="0.0" kd="1000.0" />
       </collision>
       <visual>
@@ -51,13 +44,4 @@
       </visual>
     </link>
-    <gazebo reference="${prefix}_roller_neighbor_${idx}">
-      <mu>5</mu>
-      <mu2>5</mu2>
-      <slip1>0</slip1>
-      <slip2>0</slip2>
-      <kp>5e5</kp>
-      <kd>50</kd>
-      <material>Gazebo/Grey</material>
-    </gazebo>
     <joint name="${prefix}_roller_${idx}_joint" type="continuous">
       <parent link="${parent}"/>
@@ -68,4 +52,5 @@
       <axis xyz="0 1 0"/>
       <dynamics damping="5.0" friction="1.0"/>
+      <limit effort="1.0" velocity="10"/>
     </joint>
     <joint name="${prefix}_roller_neighbor_${idx}_joint" type="continuous">
@@ -77,4 +62,5 @@
       <axis xyz="0 1 0"/>
       <dynamics damping="5.0" friction="1.0"/>
+      <limit effort="1.0" velocity="10"/>
     </joint>
   </xacro:macro>
@@ -118,26 +104,7 @@
       </collision>
     </link>
-    <gazebo reference="${prefix}_hub">
-      <surface>
-        <friction>
-          <ode>
-            <mu>1.0</mu>
-            <mu2>1.0</mu2>
-            <fdir1>0 0 0</fdir1>
-          </ode>
-        </friction>
-        <contact>
-          <ode>
-            <kp>5e5</kp>
-            <kd>50</kd>
-            <max_vel>0.01</max_vel>
-            <min_depth>0.001</min_depth>
-          </ode>
-        </contact>
-      </surface>
-    </gazebo>
     <joint name="${prefix}_joint" type="continuous">
       <parent link="${parent}"/>
-      <child link="${prefix}_hub"/>
+      <child link="${prefix}  "/>
       <origin xyz="${xyz}" rpy="${rpy}"/>
       <axis xyz="0 1 0"/>
