Commit message: correction du launcher pour le pi (les variables config n'étaient pas incluses)

File: src/car_square/model/model.xacro (robot description, xacro)
@@ -12,5 +12,5 @@
                 <collision>
                         <geometry>
-                        <box size="0.3 0.25 0.05"/>
+                        <box size="${chassis_length} ${chassis_width} ${chassis_height}"/>
                         </geometry>
                         <origin xyz="0 0 ${chassis_offset}" rpy="0 0 0"/>
@@ -18,9 +18,23 @@
                 <xacro:chassis_inertia />
         </link>
+        <link name="visual_front">
+                <visual>
+                        <geometry>
+                                <box size="${chassis_length/8} ${chassis_width/2} ${chassis_height/4}"/>
+                        </geometry>
+                        <origin xyz="0 0 0" rpy="0 0 0"/>
+                        <material name="green"/>
+                </visual>
+        </link>
+        <joint name="visual_front_joint" type="fixed">
+                <parent link="base_link"/>
+                <child link="visual_front"/>
+                <origin xyz="${chassis_length/2} 0 ${chassis_offset}" rpy="0 1.571 0"/>
+        </joint>
         <!-- LINKS ET JOINTS DES ROUES -->
         <xacro:omni_wheel
                 prefix="lf"
                 parent="base_link"
-                xyz="${chassis_length/2} ${chassis_width/2 + wheel_width} ${r}"
+                xyz="${chassis_length/2 + wheel_offset} ${chassis_width/2 + wheel_offset} ${r}"
                 rpy="0 0 ${-pi/4}"
         />
@@ -28,5 +42,5 @@
                 prefix="rf"
                 parent="base_link"
-                xyz="${chassis_length/2} ${-(chassis_width/2 + wheel_width)} ${r}"
+                xyz="${chassis_length/2 + wheel_offset} ${-(chassis_width/2 + wheel_offset)} ${r}"
                 rpy="0 0 ${5*pi/4}"
         />
@@ -34,5 +48,5 @@
                 prefix="lb"
                 parent="base_link"
-                xyz="${-(chassis_length/2)} ${chassis_width/2 + wheel_width} ${r}"
+                xyz="${-(chassis_length/2 + wheel_offset)} ${chassis_width/2 + wheel_offset} ${r}"
                 rpy="0 0 ${pi/4}"
         />
@@ -40,7 +54,51 @@
                 prefix="rb"
                 parent="base_link"
-                xyz="${-(chassis_length/2)} ${-(chassis_width/2 + wheel_width)} ${r}"
+                xyz="${-(chassis_length/2 + wheel_offset)} ${-(chassis_width/2 + wheel_offset)} ${r}"
                 rpy="0 0 ${-5*pi/4}"
         />
+        <!--  -->
+        <link name="mat_link">
+                <visual>
+                        <origin xyz="0 0 0" rpy="0 0 0"/>
+                        <geometry>
+                                <cylinder length="${mat_length}" radius="${mat_radius}"/>
+                        </geometry>
+                        <material name="red"/>
+                </visual>
+                <collision name="collision">
+                        <origin xyz="0 0 0" rpy="0 0 0"/>
+                        <geometry>
+                                <cylinder length="${mat_length}" radius="${mat_radius}"/>
+                        </geometry>
+                </collision>
+        </link>
+        <joint name="mat_joint" type="fixed">
+                        <origin xyz="0 0 ${chassis_offset - chassis_height/4 + mat_length/2}" rpy="0 0 0"/>
+                <parent link="base_link"/>
+                <child link="mat_link"/>
+                <axis xyz="0 1 0" rpy="0 0 0"/>
+        </joint>
+        <!-- LINKS ET JOINTS DU LIDAR -->
+        <link name="lidar_link">
+                <visual>
+                        <origin xyz="0 0 0" rpy="0 0 0"/>
+                        <geometry>
+                                <cylinder length="${lidar_length}" radius="${lidar_radius}"/>
+                        </geometry>
+                        <material name="green"/>
+                </visual>
+                <collision name="collision">
+                        <origin xyz="0 0 0" rpy="0 0 0"/>
+                        <geometry>
+                                <cylinder length="${lidar_length}" radius="${lidar_radius}"/>
+                        </geometry>
+                </collision>
+        </link>
+        <joint name="lidar_joint" type="fixed">
+                        <origin xyz="0 0 ${chassis_offset - chassis_height/4 + mat_length + lidar_length/2}" rpy="0 0 0"/>
+                <parent link="base_link"/>
+                <child link="lidar_link"/>
+                <axis xyz="0 1 0" rpy="0 0 0"/>
+        </joint>
         <!-- ROS2_CONTROL -->
         <ros2_control name="RobotController" type="system">

File: src/car_square/model/wheels/omni_wheel.urdf.xacro (robot description, xacro)
@@ -106,5 +106,5 @@
     <joint name="${prefix}_joint" type="continuous">
       <parent link="${parent}"/>
-      <child link="${prefix}  "/>
+      <child link="${prefix}_hub"/>
       <origin xyz="${xyz}" rpy="${rpy}"/>
       <axis xyz="0 1 0"/>

Commit message: Ajout d'un noeud ros permettant d'exporter les joints states de la simu dans /micro_controlller/joint_states pour utiliser le même noeud de contrôle qu'IRL

File: src/car_square/model/model.xacro (robot description, xacro)
@@ -123,10 +123,10 @@
                         <state_interface name="velocity"/>
                 </joint>
-                <joint name="lb_joint">
+                <joint name="rb_joint">
                         <command_interface name="velocity"/>
                         <state_interface name="position"/>
                         <state_interface name="velocity"/>
                 </joint>
-                <joint name="rb_joint">
+                <joint name="lb_joint">
                         <command_interface name="velocity"/>
                         <state_interface name="position"/>

File: src/car_square/model/model_simu.xacro (robot description, xacro)
@@ -112,44 +112,4 @@
                         <state_interface name="velocity"/>
                 </joint>
-                <joint name="lf_roller_0_joint">
-                        <command_interface name="velocity"/>
-                        <state_interface name="position"/>
-                        <state_interface name="velocity"/>
-                </joint>
-                <joint name="lf_roller_neighbor_0_joint">
-                        <command_interface name="velocity"/>
-                        <state_interface name="position"/>
-                        <state_interface name="velocity"/>
-                </joint>
-                <joint name="lf_roller_1_joint">
-                        <command_interface name="velocity"/>
-                        <state_interface name="position"/>
-                        <state_interface name="velocity"/>
-                </joint>
-                <joint name="lf_roller_neighbor_1_joint">
-                        <command_interface name="velocity"/>
-                        <state_interface name="position"/>
-                        <state_interface name="velocity"/>
-                </joint>
-                <joint name="lf_roller_2_joint">
-                        <command_interface name="velocity"/>
-                        <state_interface name="position"/>
-                        <state_interface name="velocity"/>
-                </joint>
-                <joint name="lf_roller_neighbor_2_joint">
-                        <command_interface name="velocity"/>
-                        <state_interface name="position"/>
-                        <state_interface name="velocity"/>
-                </joint>
-                <joint name="lf_roller_3_joint">
-                        <command_interface name="velocity"/>
-                        <state_interface name="position"/>
-                        <state_interface name="velocity"/>
-                </joint>
-                <joint name="lf_roller_neighbor_3_joint">
-                        <command_interface name="velocity"/>
-                        <state_interface name="position"/>
-                        <state_interface name="velocity"/>
-                </joint>
                 <joint name="rf_joint">
                         <command_interface name="velocity"/>
@@ -157,40 +117,5 @@
                         <state_interface name="velocity"/>
                 </joint>
-                <joint name="rf_roller_0_joint">
-                        <command_interface name="velocity"/>
-                        <state_interface name="position"/>
-                        <state_interface name="velocity"/>
-                </joint>
-                <joint name="rf_roller_neighbor_0_joint">
-                        <command_interface name="velocity"/>
-                        <state_interface name="position"/>
-                        <state_interface name="velocity"/>
-                </joint>
-                <joint name="rf_roller_1_joint">
-                        <command_interface name="velocity"/>
-                        <state_interface name="position"/>
-                        <state_interface name="velocity"/>
-                </joint>
-                <joint name="rf_roller_neighbor_1_joint">
-                        <command_interface name="velocity"/>
-                        <state_interface name="position"/>
-                        <state_interface name="velocity"/>
-                </joint>
-                <joint name="rf_roller_2_joint">
-                        <command_interface name="velocity"/>
-                        <state_interface name="position"/>
-                        <state_interface name="velocity"/>
-                </joint>
-                <joint name="rf_roller_neighbor_2_joint">
-                        <command_interface name="velocity"/>
-                        <state_interface name="position"/>
-                        <state_interface name="velocity"/>
-                </joint>
-                <joint name="rf_roller_3_joint">
-                        <command_interface name="velocity"/>
-                        <state_interface name="position"/>
-                        <state_interface name="velocity"/>
-                </joint>
-                <joint name="rf_roller_neighbor_3_joint">
+                <joint name="rb_joint">
                         <command_interface name="velocity"/>
                         <state_interface name="position"/>
@@ -202,89 +127,4 @@
                         <state_interface name="velocity"/>
                 </joint>
-                <joint name="lb_roller_0_joint">
-                        <command_interface name="velocity"/>
-                        <state_interface name="position"/>
-                        <state_interface name="velocity"/>
-                </joint>
-                <joint name="lb_roller_neighbor_0_joint">
-                        <command_interface name="velocity"/>
-                        <state_interface name="position"/>
-                        <state_interface name="velocity"/>
-                </joint>
-                <joint name="lb_roller_1_joint">
-                        <command_interface name="velocity"/>
-                        <state_interface name="position"/>
-                        <state_interface name="velocity"/>
-                </joint>
-                <joint name="lb_roller_neighbor_1_joint">
-                        <command_interface name="velocity"/>
-                        <state_interface name="position"/>
-                        <state_interface name="velocity"/>
-                </joint>
-                <joint name="lb_roller_2_joint">
-                        <command_interface name="velocity"/>
-                        <state_interface name="position"/>
-                        <state_interface name="velocity"/>
-                </joint>
-                <joint name="lb_roller_neighbor_2_joint">
-                        <command_interface name="velocity"/>
-                        <state_interface name="position"/>
-                        <state_interface name="velocity"/>
-                </joint>
-                <joint name="lb_roller_3_joint">
-                        <command_interface name="velocity"/>
-                        <state_interface name="position"/>
-                        <state_interface name="velocity"/>
-                </joint>
-                <joint name="lb_roller_neighbor_3_joint">
-                        <command_interface name="velocity"/>
-                        <state_interface name="position"/>
-                        <state_interface name="velocity"/>
-                </joint>
-                <joint name="rb_joint">
-                        <command_interface name="velocity"/>
-                        <state_interface name="position"/>
-                        <state_interface name="velocity"/>
-                </joint>
-                <joint name="rb_roller_0_joint">
-                        <command_interface name="velocity"/>
-                        <state_interface name="position"/>
-                        <state_interface name="velocity"/>
-                </joint>
-                <joint name="rb_roller_neighbor_0_joint">
-                        <command_interface name="velocity"/>
-                        <state_interface name="position"/>
-                        <state_interface name="velocity"/>
-                </joint>
-                <joint name="rb_roller_1_joint">
-                        <command_interface name="velocity"/>
-                        <state_interface name="position"/>
-                        <state_interface name="velocity"/>
-                </joint>
-                <joint name="rb_roller_neighbor_1_joint">
-                        <command_interface name="velocity"/>
-                        <state_interface name="position"/>
-                        <state_interface name="velocity"/>
-                </joint>
-                <joint name="rb_roller_2_joint">
-                        <command_interface name="velocity"/>
-                        <state_interface name="position"/>
-                        <state_interface name="velocity"/>
-                </joint>
-                <joint name="rb_roller_neighbor_2_joint">
-                        <command_interface name="velocity"/>
-                        <state_interface name="position"/>
-                        <state_interface name="velocity"/>
-                </joint>
-                <joint name="rb_roller_3_joint">
-                        <command_interface name="velocity"/>
-                        <state_interface name="position"/>
-                        <state_interface name="velocity"/>
-                </joint>
-                <joint name="rb_roller_neighbor_3_joint">
-                        <command_interface name="velocity"/>
-                        <state_interface name="position"/>
-                        <state_interface name="velocity"/>
-                </joint>
         </ros2_control>
 </robot>
