Commit message: ajout d'un contrôle de la position

File: src/car_square/model/wheels/omni_wheel.urdf.xacro (robot description, xacro)
@@ -6,6 +6,6 @@
     <link name="${prefix}_roller_${idx}">
       <inertial>
-        <mass value="9.1"/>
-        <inertia ixx="0.0812" iyy="0.0812" izz="0.0473" ixy="0" ixz="0" iyz="0"/>
+        <mass value="0.1"/>
+        <inertia ixx="10" iyy="10" izz="10" ixy="0" ixz="0" iyz="0"/>
       </inertial>
       <collision>
@@ -24,25 +24,16 @@
     </link>
     <gazebo reference="${prefix}_roller_${idx}">
-      <surface>
-        <friction>
-          <ode>
-            <mu>1.0</mu>
-            <mu2>1.0</mu2>
-          </ode>
-        </friction>
-        <contact>
-          <ode>
-            <kp>1e+5</kp>
-            <kd>100.0</kd>
-            <max_vel>0.01</max_vel>
-            <min_depth>0</min_depth>
-          </ode>
-        </contact>
-      </surface>
+      <mu>1</mu>
+      <mu2>1</mu2>
+      <slip1>0</slip1>
+      <slip2>0</slip2>
+      <kp>1e+13</kp>  <!-- Rigidité très élevée -->
+      <kd>1.0</kd>
+      <material>Gazebo/Grey</material>
     </gazebo>
     <link name="${prefix}_roller_neighbor_${idx}">
       <inertial>
-        <mass value="9.1"/>
-        <inertia ixx="0.0812" iyy="0.0812" izz="0.0473" ixy="0" ixz="0" iyz="0"/>
+        <mass value="0.1"/>
+        <inertia ixx="10" iyy="10" izz="10" ixy="0" ixz="0" iyz="0"/>
       </inertial>
       <collision>
@@ -61,20 +52,11 @@
     </link>
     <gazebo reference="${prefix}_roller_neighbor_${idx}">
-      <surface>
-        <friction>
-          <ode>
-            <mu>1.0</mu>
-            <mu2>1.0</mu2>
-          </ode>
-        </friction>
-        <contact>
-          <ode>
-            <kp>1e+5</kp>
-            <kd>100.0</kd>
-            <max_vel>0.01</max_vel>
-            <min_depth>0</min_depth>
-          </ode>
-        </contact>
-      </surface>
+      <mu>1</mu>
+      <mu2>1</mu2>
+      <slip1>0</slip1>
+      <slip2>0</slip2>
+      <kp>1e+13</kp>  <!-- Rigidité très élevée -->
+      <kd>1.0</kd>
+      <material>Gazebo/Grey</material>
     </gazebo>
     <joint name="${prefix}_roller_${idx}_joint" type="continuous">
@@ -85,5 +67,5 @@
         rpy="${3*pi/2 - angle1} 0 1.5708"/>
       <axis xyz="0 1 0"/>
-      <dynamics damping="0.01" friction="0.0"/>
+      <dynamics damping="0.0" friction="0.0"/>
     </joint>
     <joint name="${prefix}_roller_neighbor_${idx}_joint" type="continuous">
@@ -94,5 +76,5 @@
         rpy="${3*pi/2 - angle2} 0 1.5708"/>
       <axis xyz="0 1 0"/>
-      <dynamics damping="0.01" friction="0.0"/>
+      <dynamics damping="0.0" friction="0.0"/>
     </joint>
   </xacro:macro>
@@ -120,5 +102,5 @@
         <origin rpy="1.5708 0 0"/>
         <mass value="66.86064"/>
-        <inertia ixx="3.009" iyy="2.1239" izz="2.1239" ixy="0.0" ixz="0.0" iyz="0.0"/>
+        <inertia ixx="0.009" iyy="0.1239" izz="0.1239" ixy="0.0" ixz="0.0" iyz="0.0"/>
       </inertial>
       <visual>
@@ -147,8 +129,8 @@
         <contact>
           <ode>
-            <kp>1e+5</kp>
+            <kp>1e+6</kp>
             <kd>100.0</kd>
             <max_vel>0.01</max_vel>
-            <min_depth>0</min_depth>
+            <min_depth>0.001</min_depth>
           </ode>
         </contact>
@@ -160,5 +142,5 @@
       <origin xyz="${xyz}" rpy="${rpy}"/>
       <axis xyz="0 1 0"/>
-      <dynamics damping="0.0" friction="0.0"/>
+      <dynamics damping="0.5" friction="0.1"/>
     </joint>
     <xacro:roller_loop
